File: power.kicad_sch (KiCad schematic)
At the start: 25 parts, among them J3 EXT_PWR, J4 V_ORBITTY, J5 V_HUB, J6 PWR_SWITCH, Q2 Q_PMOS_GDS, U1 TL7702A, U5 P783F-Q24-S5-S

Commit message: Possible revision without feedback. Changes on schematic but not PCB.
Parts:
- removed R2: 50k, Resistor_SMD:R_1206_3216Metric_Pad1.30x1.75mm_HandSolder, symbol Device:R_US
- removed R3: 1M, Resistor_SMD:R_1206_3216Metric_Pad1.30x1.75mm_HandSolder, symbol Device:R_US
- added R?: 50k, symbol Device:R_US
Connections:
- net GND: now also R?.2
- net POWEROFF_OD: now also R?.1
Changed lines of the file:
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@@
 (kicad_sch (version 20211123) (generator eeschema)
   (paper "A4")
-  (junction (at 130.81 31.75) (diameter 0) (color 0 0 0 0)
-  )
-  (junction (at 140.97 46.99) (diameter 0) (color 0 0 0 0)
-  )
   (junction (at 168.91 31.75) (diameter 0) (color 0 0 0 0)
   )
@@
   (junction (at 76.2 121.92) (diameter 0) (color 0 0 0 0)
   )
+  (junction (at 109.22 140.97) (diameter 0) (color 0 0 0 0)
+  )
   (junction (at 161.29 74.93) (diameter 0) (color 0 0 0 0)
   )
@@
   )
   (junction (at 191.77 59.69) (diameter 0) (color 0 0 0 0)
-  )
-  (junction (at 49.53 133.35) (diameter 0) (color 0 0 0 0)
   )
   (junction (at 57.15 156.21) (diameter 0) (color 0 0 0 0)
@@
     (stroke (width 0) (type default) (color 0 0 0 0))
   )
-  (wire (pts (xy 140.97 46.99) (xy 140.97 39.37))
+  (wire (pts (xy 140.97 39.37) (xy 140.97 57.15))
     (stroke (width 0) (type default) (color 0 0 0 0))
   )
@@
     (stroke (width 0) (type default) (color 0 0 0 0))
   )
+  (wire (pts (xy 109.22 152.4) (xy 109.22 156.21))
+    (stroke (width 0) (type default) (color 0 0 0 0))
+  )
   (wire (pts (xy 177.8 36.83) (xy 177.8 34.29))
     (stroke (width 0) (type default) (color 0 0 0 0))
@@
     (stroke (width 0) (type default) (color 0 0 0 0))
   )
+  (wire (pts (xy 109.22 140.97) (xy 109.22 144.78))
+    (stroke (width 0) (type default) (color 0 0 0 0))
+  )
   (wire (pts (xy 168.91 31.75) (xy 168.91 33.02))
     (stroke (width 0) (type default) (color 0 0 0 0))
@@
     (stroke (width 0) (type default) (color 0 0 0 0))
   )
-  (wire (pts (xy 95.25 156.21) (xy 107.95 156.21))
+  (wire (pts (xy 95.25 156.21) (xy 109.22 156.21))
     (stroke (width 0) (type default) (color 0 0 0 0))
   )
@@
     (stroke (width 0) (type default) (color 0 0 0 0))
   )
-  (wire (pts (xy 130.81 46.99) (xy 140.97 46.99))
-    (stroke (width 0) (type default) (color 0 0 0 0))
-  )
-  (wire (pts (xy 48.26 133.35) (xy 49.53 133.35))
-    (stroke (width 0) (type default) (color 0 0 0 0))
-  )
-  (wire (pts (xy 26.67 133.35) (xy 40.64 133.35))
-    (stroke (width 0) (type default) (color 0 0 0 0))
-  )
   (wire (pts (xy 233.68 46.99) (xy 233.68 49.53))
     (stroke (width 0) (type default) (color 0 0 0 0))
@@
     (stroke (width 0) (type default) (color 0 0 0 0))
   )
-  (wire (pts (xy 130.81 36.83) (xy 130.81 31.75))
-    (stroke (width 0) (type default) (color 0 0 0 0))
-  )
-  (wire (pts (xy 130.81 44.45) (xy 130.81 46.99))
-    (stroke (width 0) (type default) (color 0 0 0 0))
-  )
   (polyline (pts (xy 87.63 90.17) (xy 87.63 15.24))
     (stroke (width 0) (type default) (color 0 0 0 0))
@@
     (stroke (width 0) (type default) (color 0 0 0 0))
   )
-  (wire (pts (xy 130.81 31.75) (xy 135.89 31.75))
-    (stroke (width 0) (type default) (color 0 0 0 0))
-  )
   (wire (pts (xy 213.36 38.1) (xy 213.36 40.64))
     (stroke (width 0) (type default) (color 0 0 0 0))
@@
     (stroke (width 0) (type default) (color 0 0 0 0))
   )
-  (wire (pts (xy 140.97 57.15) (xy 140.97 46.99))
-    (stroke (width 0) (type default) (color 0 0 0 0))
-  )
   (polyline (pts (xy 90.17 15.24) (xy 281.94 15.24))
     (stroke (width 0) (type default) (color 0 0 0 0))
@@
     (stroke (width 0) (type default) (color 0 0 0 0))
   )
-  (wire (pts (xy 125.73 31.75) (xy 130.81 31.75))
+  (wire (pts (xy 125.73 31.75) (xy 135.89 31.75))
     (stroke (width 0) (type default) (color 0 0 0 0))
   )
@@
   )
   (text "72mW max dissipation at 3A load" (at 125.73 19.05 0)
-    (effects (font (size 1.27 1.27)) (justify left bottom))
-  )
-  (label "POWEROFF_OD" (at 26.67 133.35 0)
     (effects (font (size 1.27 1.27)) (justify left bottom))
   )
@@
     (pin "2")
   )
-  (symbol (lib_id "Connector_Generic:Conn_01x02") (at 36.83 46.99 180)
+  (symbol (lib_id "Connector_Generic:Conn_01x02") (at 36.83 46.99 180) (unit 1)
     (in_bom yes) (on_board yes)
     (property "Reference" "J3" (id 0) (at 34.798 46.7868 0)
@@
     )
     (property "Datasheet" "~" (id 3) (at 36.83 34.29 0)
-      (effects (font (size 1.27 1.27)) hide)
-    )
-    (pin "1")
-    (pin "2")
-  )
-  (symbol (lib_id "Device:R_US") (at 130.81 40.64 0) (unit 1)
-    (in_bom yes) (on_board yes)
-    (property "Reference" "R2" (id 0) (at 132.5372 39.4716 0)
-      (effects (font (size 1.27 1.27)) (justify left))
-    )
-    (property "Value" "50k" (id 1) (at 132.5372 41.783 0)
-      (effects (font (size 1.27 1.27)) (justify left))
-    )
-    (property "Footprint" "Resistor_SMD:R_1206_3216Metric_Pad1.30x1.75mm_HandSolder" (id 2) (at 131.826 40.894 90)
-      (effects (font (size 1.27 1.27)) hide)
-    )
-    (property "Datasheet" "~" (id 3) (at 130.81 40.64 0)
       (effects (font (size 1.27 1.27)) hide)
     )
@@
     (pin "2")
   )
-  (symbol (lib_id "Device:R_US") (at 44.45 133.35 90) (unit 1)
-    (in_bom yes) (on_board yes)
-    (property "Reference" "R3" (id 0) (at 44.45 128.143 90))
-    (property "Value" "1M" (id 1) (at 44.45 130.4544 90))
-    (property "Footprint" "Resistor_SMD:R_1206_3216Metric_Pad1.30x1.75mm_HandSolder" (id 2) (at 44.704 132.334 90)
-      (effects (font (size 1.27 1.27)) hide)
-    )
-    (property "Datasheet" "~" (id 3) (at 44.45 133.35 0)
-      (effects (font (size 1.27 1.27)) hide)
-    )
-    (pin "1")
-    (pin "2")
-  )
   (symbol (lib_id "power:+12V") (at 31.75 64.77 0) (mirror y) (unit 1)
     (in_bom yes) (on_board yes)
@@
     (pin "1")
   )
+  (symbol (lib_id "Device:R_US") (at 109.22 148.59 0) (unit 1)
+    (in_bom yes) (on_board yes) (fields_autoplaced)
+    (property "Reference" "R?" (id 0) (at 111.76 147.3199 0)
+      (effects (font (size 1.27 1.27)) (justify left))
+    )
+    (property "Value" "50k" (id 1) (at 111.76 149.8599 0)
+      (effects (font (size 1.27 1.27)) (justify left))
+    )
+    (property "Footprint" "" (id 2) (at 110.236 148.844 90)
+      (effects (font (size 1.27 1.27)) hide)
+    )
+    (property "Datasheet" "~" (id 3) (at 109.22 148.59 0)
+      (effects (font (size 1.27 1.27)) hide)
+    )
+    (pin "1")
+    (pin "2")
+  )
 )

Commit message: Rev 3 Changes
Parts:
- removed C2: 100n, Capacitor_SMD:C_1206_3216Metric_Pad1.33x1.80mm_HandSolder, symbol Device:C
- removed R?: 50k, symbol Device:R_US
- removed U1: TL7702A, Package_SO:SOIC-8_3.9x4.9mm_P1.27mm, symbol Power_Supervisor:TL7702A
- added C2: 1000u, Capacitor_THT:CP_Radial_D13.0mm_P5.00mm, symbol Device:C_Polarized_US
- added Q3: 2N7002, Package_TO_SOT_SMD:SOT-23, symbol Transistor_FET:2N7002
- added R11, R6: 50k, Resistor_SMD:R_1206_3216Metric_Pad1.30x1.75mm_HandSolder, symbol Device:R_US
- added R2: 10M, Resistor_SMD:R_1206_3216Metric_Pad1.30x1.75mm_HandSolder, symbol Device:R_US
- added R3: 870k, Resistor_SMD:R_1206_3216Metric_Pad1.30x1.75mm_HandSolder, symbol Device:R_US
- added U1: NCP711, Package_TO_SOT_SMD:SOT-23-5, symbol Customs:NCP711
- added U2: MIC2779L, Package_TO_SOT_SMD:SOT-23-5, symbol Customs:MIC2779L
- C1: value 10n -> 1u
- C29: footprint Capacitor_THT:CP_Radial_D5.0mm_P2.00mm -> Capacitor_THT:CP_Radial_D8.0mm_P3.50mm
- C3: value 100n -> 1u
- R4: value 102k -> 12k
- R5: value 34.8k -> 118k
Connections:
- net GND: now also C2.2, Q3.2 (S), R2.2, R6.2, U1.2 (GND), U2.2 (GND)
- net POWEROFF_OD: now also Q3.3 (D), R11.2
- net Vext: now also R11.1, R3.1, U1.1 (IN); no longer R4.1
- net at F1.2, J6.2 (Pin_2): now also C2.1, R2.1
- net +3V3: now reaches C3.1
- net +3V3: now also U1.5 (OUT), U2.5 (Vdd)
- net at R4.2, R5.1: now also U2.1 (HTH)
- new net: Q3.1 (G), R6.1, U2.4 (RST_n)
- new net: R3.2, R4.1, U2.3 (LTH)
Other:
- note added: "Thresholds: 9.5v - 10.5v 1% resistors here"
- note removed: "10v Threshold (0.3v Hysteresis)"

Commit message: Some footprint fixes.
Parts:
- removed Q3: 2N7002, Package_TO_SOT_SMD:SOT-23, symbol Transistor_FET:2N7002
- added Q3: Q_NMOS_GSD, Package_TO_SOT_SMD:SOT-23_Handsoldering, symbol Device:Q_NMOS_GSD
Connections:
- net GND: now also Q3.2 (S)
- net POWEROFF_OD: now also Q3.3 (D)
- net at R6.1, U2.4 (RST_n): now also Q3.1 (G)
Changed lines of the file:
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@@
     (pin "1")
-  )
-  (symbol (lib_id "Transistor_FET:2N7002") (at 123.19 128.27 0) (unit 1)
-    (in_bom yes) (on_board yes) (fields_autoplaced)
-    (property "Reference" "Q3" (id 0) (at 129.54 126.9999 0)
-      (effects (font (size 1.27 1.27)) (justify left))
-    )
-    (property "Value" "2N7002" (id 1) (at 129.54 129.5399 0)
-      (effects (font (size 1.27 1.27)) (justify left))
-    )
-    (property "Footprint" "Package_TO_SOT_SMD:SOT-23" (id 2) (at 128.27 130.175 0)
-      (effects (font (size 1.27 1.27) italic) (justify left) hide)
-    )
-    (property "Datasheet" "https://www.onsemi.com/pub/Collateral/NDS7002A-D.PDF" (id 3) (at 123.19 128.27 0)
-      (effects (font (size 1.27 1.27)) (justify left) hide)
-    )
-    (pin "1")
-    (pin "2")
-    (pin "3")
   )
   (symbol (lib_id "power:GND") (at 76.2 144.78 0) (unit 1)
@@
     (pin "1")
   )
+  (symbol (lib_id "Device:Q_NMOS_GSD") (at 123.19 128.27 0) (unit 1)
+    (in_bom yes) (on_board yes)
+    (property "Reference" "Q3" (id 0) (at 128.397 127.1016 0)
+      (effects (font (size 1.27 1.27)) (justify left))
+    )
+    (property "Value" "Q_NMOS_GSD" (id 1) (at 128.397 129.413 0)
+      (effects (font (size 1.27 1.27)) (justify left))
+    )
+    (property "Footprint" "Package_TO_SOT_SMD:SOT-23_Handsoldering" (id 2) (at 128.27 125.73 0)
+      (effects (font (size 1.27 1.27)) hide)
+    )
+    (property "Datasheet" "~" (id 3) (at 123.19 128.27 0)
+      (effects (font (size 1.27 1.27)) hide)
+    )
+    (pin "1")
+    (pin "2")
+    (pin "3")
+  )
   (symbol (lib_id "Device:R_US") (at 114.3 133.35 0) (unit 1)

Commit message: Changed to axial capacitor, fixed mounting hole size.
Parts:
- C2: footprint Capacitor_THT:CP_Radial_D13.0mm_P5.00mm -> Capacitor_THT:CP_Axial_L30.0mm_D12.5mm_P35.00mm_Horizontal
Changed lines of the file:
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@@
       (effects (font (size 1.27 1.27)) (justify left))
     )
-    (property "Footprint" "Capacitor_THT:CP_Radial_D13.0mm_P5.00mm" (id 2) (at 52.07 45.72 0)
+    (property "Footprint" "Capacitor_THT:CP_Axial_L30.0mm_D12.5mm_P35.00mm_Horizontal" (id 2) (at 52.07 45.72 0)
       (effects (font (size 1.27 1.27)) hide)
     )
